File: HDK/mecatron-power-distribution-unit.kicad_sch (KiCad schematic)
At the start: 18 parts, among them J101 PwrIn_{1}, J102 PwrIn_{2}, J103 PwrOut_{1}, J104 PwrOut_{1}, J105 PwrOut_{1}, J106 PwrOut_{1}, J107 PwrOut_{1}, J108 PwrOut_{1}, J109 PwrOut_{1}, J110 PwrOut_{1}, K101 Relay_SPDT, K102 Relay_SPDT, SW101 E-STOP, SW102 PwrSw

Commit message: added working v1
Parts:
- removed J105, J106, J107, J108, J109, J110: PwrOut_{1}, Connector_Molex:Molex_Mini-Fit_Jr_5566-02A_2x01_P4.20mm_Vertical, symbol Connector_Generic:Conn_01x02
- removed SW101: E-STOP, symbol Switch:SW_SPST
- removed SW102: PwrSw, symbol Switch:SW_SPST
- J103: value PwrOut_{1} -> PwrSw; footprint Connector_Molex:Molex_Mini-Fit_Jr_5566-02A_2x01_P4.20mm_Vertical -> (none)
- J104: value PwrOut_{1} -> E-Stop; footprint Connector_Molex:Molex_Mini-Fit_Jr_5566-02A_2x01_P4.20mm_Vertical -> (none)
- renumbered D102 to D101, D101 to D102, F102 to F101, F101 to F102, K102 to K101, K101 to K102
Connections:
- net GND: no longer J103.2 (Pin_2), J104.2 (Pin_2)
- net VCCF_{1}: no longer J103.1 (Pin_1), J104.1 (Pin_1)
- net VCC_{2}: now also J104.1 (Pin_1)
- net at D102.1 (K), K102.A1: now also J104.2 (Pin_2)
- net at F101.2, K101.12: now also J103.1 (Pin_1)
- net at D101.1 (K), K101.A1: now also J103.2 (Pin_2)
Other:
- added sheet PwrOut1 (PwrOut1.kicad_sch)
- added sheet PwrOut2 (PwrOut2.kicad_sch)
- note added: "Assume e-stop cuts only propulsion & actuators"
- note added: "Power Control"
- note added: "Proposed Future features: 1. Over & Under & Reverse & Voltage & Short Circuit Protection 2. Power Meter in-built 3. Relay protection (via optocoupler) 4. Allow VCC1 to be on/off by mcu too"
- note added: "Q: Assume VCC_{2} powers relay switch? Without it, powering on propulsion is useless"
- note removed: "Assume e-stop cuts only thrusters and actuators"
- note removed: "Power Connectors (thrust & actuators)"
- note removed: "PwrOut connectors: (XT60) Currect Max: 30A (Cont)"
- moved on the sheet: D101, D102, F101, F102, J101, J102, K101, K102

Commit message: updated sch
Parts:
- D101: renamed from D102; footprint (none) -> Diode_SMD:D_SMA
- D102: renamed from D101; footprint (none) -> Diode_SMD:D_SMA
- J103: renamed from J104; footprint (none) -> Connector_JST:JST_XH_B2B-XH-AM_1x02_P2.50mm_Vertical
- J104: renamed from J103; footprint (none) -> Connector_JST:JST_XH_B2B-XH-AM_1x02_P2.50mm_Vertical
- renumbered K102 to K101, K101 to K102
Connections:
- net VCC_{1}: no longer J101.1 (Pin_1)
- net VCC_{2}: no longer J102.1 (Pin_1)
- new net VCC_{Main}: J101.1 (Pin_1)
- new net VCC_{Sec}: J102.1 (Pin_1)
Other:
- note removed: "Q: Assume VCC_{2} powers relay switch? Without it, powering on propulsion is useless"
- moved on the sheet: J101, J102

Commit message: added connectors
Parts:
- D101, D102: value D -> 1N4004; footprint Diode_SMD:D_SMA -> Diode_THT:D_DO-41_SOD81_P7.62mm_Horizontal
- J101, J102: footprint Connector_AMASS:AMASS_XT60-F_1x02_P7.20mm_Vertical -> mecatron-kicad-footprints:AMASS_XT60PW-M_1x02_P7.20mm_Horizontal
Changed lines of the file:
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@@
 			)
 		)
-		(property "Footprint" "Connector_AMASS:AMASS_XT60-F_1x02_P7.20mm_Vertical"
+		(property "Footprint" "mecatron-kicad-footprints:AMASS_XT60PW-M_1x02_P7.20mm_Horizontal"
 			(at 39.37 31.75 0)
 			(effects
@@
 			)
 		)
-		(property "Value" "D"
+		(property "Value" "1N4004"
 			(at 133.35 59.69 0)
 			(effects
@@
 			)
 		)
-		(property "Footprint" "Diode_SMD:D_SMA"
+		(property "Footprint" "Diode_THT:D_DO-41_SOD81_P7.62mm_Horizontal"
 			(at 133.35 63.5 0)
 			(effects
@@
 			)
 		)
-		(property "Footprint" "Connector_AMASS:AMASS_XT60-F_1x02_P7.20mm_Vertical"
+		(property "Footprint" "mecatron-kicad-footprints:AMASS_XT60PW-M_1x02_P7.20mm_Horizontal"
 			(at 39.37 24.13 0)
 			(effects
@@
 			)
 		)
-		(property "Value" "D"
+		(property "Value" "1N4004"
 			(at 58.42 59.69 0)
 			(effects
@@
 			)
 		)
-		(property "Footprint" "Diode_SMD:D_SMA"
+		(property "Footprint" "Diode_THT:D_DO-41_SOD81_P7.62mm_Horizontal"
 			(at 58.42 63.5 0)
 			(effects
