File: HV/MecatronPDU-HV.kicad_pcb (KiCad board)
At the start: 2 copper layers, 80 x 80 mm, 35 parts, among them J101 Power In, J102 V_{Comp}, J106 E-Stops, J201 Power Out, J202 Power Out, J203 Power Out, J204 Power Out, J205 Power Out, J206 Power Out, J207 Power Out, J208 Power Out, J209 Power Out, K101 Relay_SPST-NO

Commit message: final HV
Parts:
- removed REF** (x2): Symbol_HighVoltage_Triangle_6x6mm_Copper, Symbol:Symbol_HighVoltage_Triangle_6x6mm_Copper
- added D102: LED, LED_THT:LED_D5.0mm_Clear, F.Cu at (125.5, 97.5)
- added D103: LED, LED_THT:LED_D5.0mm_Clear, F.Cu at (125.5, 87.0)
- added D104: LED, LED_THT:LED_D5.0mm_Clear, F.Cu at (125.5, 76.5)
- added G***: LOGO, mecatron-logo-fp:mecatron-logo-fp30, F.Cu at (96.0, 123.5)
- added G***: LOGO, mecatron-logo-fp:mecatron-logo-fp30, B.Cu at (96.0, 123.5)
- added R101: 1k, Resistor_THT:R_Axial_DIN0204_L3.6mm_D1.6mm_P5.08mm_Horizontal, F.Cu at (123.0, 104.0)
- added R102: 1k, Resistor_THT:R_Axial_DIN0204_L3.6mm_D1.6mm_P5.08mm_Horizontal, F.Cu at (118.0, 104.0)
- added R103: 1k, Resistor_THT:R_Axial_DIN0204_L3.6mm_D1.6mm_P5.08mm_Horizontal, F.Cu at (120.5, 104.0)
- C101, C102, C103, C104, C105, C201, C202, C203, C204, C205, C206, C207, C208, C209: footprint scottcjx-kicad-lib:CP_Radial_D10.0mm_P5.00mm -> Capacitor_THT:CP_Radial_D10.0mm_P5.00mm
- J101: footprint Connector_AMASS:AMASS_XT60-M_1x02_P7.20mm_Vertical -> Connector_AMASS:AMASS_XT60PW-M_1x02_P7.20mm_Horizontal
- moved J102 23.6 mm to (110.5, 109.5)
- moved J106 20.2 mm to (113.0, 115.7), turned to -90 degrees
- moved D101 13.2 mm to (86.0, 101.5)
- moved K101 12.4 mm to (96.1, 109.9)
- moved F101 12.1 mm to (72.0, 106.0), turned to 0 degrees
- moved J101 6.71 mm to (76.5, 113.0), turned to 180 degrees
- moved C101 2.51 mm to (59.5, 113.0)
- moved C102 2.51 mm to (59.5, 101.5)
- moved C103 2.50 mm to (59.5, 90.1)
- moved C104 2.50 mm to (59.5, 78.5)
- moved C105 2.50 mm to (59.5, 67.0)
- moved C204 2.45 mm to (77.0, 80.0)
- moved C205 2.45 mm to (94.0, 80.0)
- moved C206 2.45 mm to (111.0, 80.0)
- moved C207 2.45 mm to (77.0, 95.0)
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Connections:
- net Net-(D101-K) renamed /relay_sig
Routing:
- net VCC: track 0.00 -> 81.6 mm
- net /relay_sig: track 33.3 -> 72.2 mm
- net Net-(D104-K): track 0.00 -> 32.7 mm
- net V_{Comp}: track 7.99 -> 34.5 mm
- net Net-(D103-K): track 0.00 -> 20.7 mm
- net Net-(D102-K): track 0.00 -> 7.50 mm
- net GND: track 0.02 -> 0.00 mm, vias 0 -> 3
Other:
- board text added: "Relay"
- board text added: "Scott CJX"
- board text added: "VCC"
- board text added: "VComp"
