File: HV/Outputs.kicad_sch (KiCad schematic)
At the start: 18 parts, among them J201 Power Out, J202 Power Out, J203 Power Out, J204 Power Out, J205 Power Out, J206 Power Out, J207 Power Out, J208 Power Out, J209 Power Out

Commit message: final HV
Parts:
- C201, C202, C203, C204, C205, C206, C207, C208, C209: footprint scottcjx-kicad-lib:CP_Radial_D10.0mm_P5.00mm -> Capacitor_THT:CP_Radial_D10.0mm_P5.00mm
Changed lines of the file:
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@@
 			)
 		)
-		(property "Footprint" "scottcjx-kicad-lib:CP_Radial_D10.0mm_P5.00mm"
+		(property "Footprint" "Capacitor_THT:CP_Radial_D10.0mm_P5.00mm"
 			(at 82.8548 31.75 0)
 			(effects
@@
 			)
 		)
-		(property "Footprint" "scottcjx-kicad-lib:CP_Radial_D10.0mm_P5.00mm"
+		(property "Footprint" "Capacitor_THT:CP_Radial_D10.0mm_P5.00mm"
 			(at 71.4248 31.75 0)
 			(effects
@@
 			)
 		)
-		(property "Footprint" "scottcjx-kicad-lib:CP_Radial_D10.0mm_P5.00mm"
+		(property "Footprint" "Capacitor_THT:CP_Radial_D10.0mm_P5.00mm"
 			(at 25.7048 31.75 0)
 			(effects
@@
 			)
 		)
-		(property "Footprint" "scottcjx-kicad-lib:CP_Radial_D10.0mm_P5.00mm"
+		(property "Footprint" "Capacitor_THT:CP_Radial_D10.0mm_P5.00mm"
 			(at 117.1448 31.75 0)
 			(effects
@@
 			)
 		)
-		(property "Footprint" "scottcjx-kicad-lib:CP_Radial_D10.0mm_P5.00mm"
+		(property "Footprint" "Capacitor_THT:CP_Radial_D10.0mm_P5.00mm"
 			(at 59.9948 31.75 0)
 			(effects
@@
 			)
 		)
-		(property "Footprint" "scottcjx-kicad-lib:CP_Radial_D10.0mm_P5.00mm"
+		(property "Footprint" "Capacitor_THT:CP_Radial_D10.0mm_P5.00mm"
 			(at 48.5648 31.75 0)
 			(effects
@@
 			)
 		)
-		(property "Footprint" "scottcjx-kicad-lib:CP_Radial_D10.0mm_P5.00mm"
+		(property "Footprint" "Capacitor_THT:CP_Radial_D10.0mm_P5.00mm"
 			(at 94.2848 31.75 0)
 			(effects
@@
 			)
 		)
-		(property "Footprint" "scottcjx-kicad-lib:CP_Radial_D10.0mm_P5.00mm"
+		(property "Footprint" "Capacitor_THT:CP_Radial_D10.0mm_P5.00mm"
 			(at 37.1348 31.75 0)
 			(effects
@@
 			)
 		)
-		(property "Footprint" "scottcjx-kicad-lib:CP_Radial_D10.0mm_P5.00mm"
+		(property "Footprint" "Capacitor_THT:CP_Radial_D10.0mm_P5.00mm"
 			(at 105.7148 31.75 0)
 			(effects
