File: LV/MecatronPDU-LV.kicad_pcb (KiCad board)
At the start: 2 copper layers, 100 x 100 mm, 21 parts, among them J101 Power In, J102 PwrSw, J103 PwrSw, K101 Relay_SPST-NO, U201 TPS5460 康威科技, U202 TPS5460 康威科技, U203 TPS5460 康威科技, U204 TPS5460 康威科技

Commit message: added lv
Parts:
- removed C201, C202, C203, C204, C205, C206, C207, C208: 560u, scottcjx-kicad-lib:CP_Radial_D10.0mm_P5.00mm
- removed J103: PwrSw, scottcjx-kicad-lib:JST_XH_B2B-XH-AM_1x02_P2.50mm_Vertical
- added C101: 560u, Capacitor_THT:CP_Radial_D10.0mm_P5.00mm, F.Cu at (59.0, 101.9)
- added C102: 560u, Capacitor_THT:CP_Radial_D10.0mm_P5.00mm, F.Cu at (70.5, 101.9)
- added C103: 560u, Capacitor_THT:CP_Radial_D10.0mm_P5.00mm, F.Cu at (59.0, 90.8)
- added C104: 560u, Capacitor_THT:CP_Radial_D10.0mm_P5.00mm, F.Cu at (70.5, 90.8)
- added C105: 560u, Capacitor_THT:CP_Radial_D10.0mm_P5.00mm, F.Cu at (59.0, 79.8)
- added C106: 560u, Capacitor_THT:CP_Radial_D10.0mm_P5.00mm, F.Cu at (70.5, 79.8)
- added C107: 560u, Capacitor_THT:CP_Radial_D10.0mm_P5.00mm, F.Cu at (59.0, 68.8)
- added C108: 560u, Capacitor_THT:CP_Radial_D10.0mm_P5.00mm, F.Cu at (70.5, 68.8)
- added D101: D, Diode_THT:D_DO-35_SOD27_P7.62mm_Horizontal, F.Cu at (60.5, 120.8)
- added G***: LOGO, mecatron-logo-fp:mecatron-logo-fp30, F.Cu at (75.0, 54.0)
- added J201: V_{HV}, Connector_JST:JST_XH_B2B-XH-AM_1x02_P2.50mm_Vertical, F.Cu at (123.2, 132.1)
- added J202: V, Connector_PinHeader_2.54mm:PinHeader_2x05_P2.54mm_Vertical, F.Cu at (123.2, 101.6)
- added J203: V, Connector_PinHeader_2.54mm:PinHeader_2x05_P2.54mm_Vertical, F.Cu at (123.2, 81.3)
- added J204: V, Connector_PinHeader_2.54mm:PinHeader_2x05_P2.54mm_Vertical, F.Cu at (123.2, 116.8)
- added J205: V_{SBC}, Connector_AMASS:AMASS_XT30UPB-M_1x02_P5.0mm_Vertical, F.Cu at (124.5, 73.6)
- J101: footprint Connector_AMASS:AMASS_XT60-M_1x02_P7.20mm_Vertical -> Connector_AMASS:AMASS_XT60PW-M_1x02_P7.20mm_Horizontal
- J102: value PwrSw -> E-Stops; footprint scottcjx-kicad-lib:JST_XH_B2B-XH-AM_1x02_P2.50mm_Vertical -> Connector_PinHeader_2.54mm:PinHeader_2x03_P2.54mm_Vertical
- moved J101 67.4 mm to (72.6, 132.8), turned to 180 degrees
- moved F101 43.5 mm to (69.5, 126.0), turned to 0 degrees
- moved U201 33.6 mm to (109.8, 78.0), turned to 90 degrees
- moved U204 33.2 mm to (109.8, 121.8), turned to -90 degrees
- moved H102 20.0 mm to (125.0, 55.0)
- moved H104 20.0 mm to (125.0, 145.0)
- moved U203 16.9 mm to (88.5, 78.0), turned to 90 degrees
- moved U202 16.9 mm to (88.5, 121.8), turned to -90 degrees
- moved K101 14.0 mm to (69.5, 114.0), turned to 90 degrees
- moved J102 9.50 mm to (53.5, 115.5)
- renumbered U203 to U201, U204 to U202, U201 to U203, U202 to U204
Connections:
- U201 pad 2: +9V -> V_{SBC}
- U202 pad 2: +12V -> +5V
- U203 pad 2: V_{SBC} -> +9V
- U204 pad 2: +5V -> +12V
Routing:
- net Net-(J102-Pin_2): track 8.84 -> 2.54 mm
- net /VCC_FUSE: track 11.6 -> 17.3 mm
- net Net-(D101-K): track 19.3 -> 22.8 mm
- net Net-(J102-Pin_3): track 0.00 -> 2.54 mm
- added copper zone on F.Cu, net +12V
- added copper zone on F.Cu, net +9V
- added copper zone on F.Cu, net V_{SBC}
- removed copper zone on B.Cu, net /VCC_FUSE
Other:
- board size 100 x 100 mm -> 80 x 100 mm
- board text added: "POWER DISTRIBUTION UNIT LV R1"
- board text added: "Scott CJX"
