File: LV/MecatronPDU-LV.kicad_sch (KiCad schematic)
At the start: 11 parts, among them J101 Power In, J102 PwrSw, J103 PwrSw, K101 Relay_SPST-NO

Commit message: added lv
Parts:
- removed D102: D_Zener, symbol Device:D_Zener
- removed J102, J103: PwrSw, scottcjx-kicad-lib:JST_XH_B2B-XH-AM_1x02_P2.50mm_Vertical, symbol Connector_Generic:Conn_01x02
- added C101, C102, C103, C104, C105, C106, C107, C108: 560u, Capacitor_THT:CP_Radial_D10.0mm_P5.00mm, symbol Device:C_Polarized
- added J102: E-Stops, Connector_PinHeader_2.54mm:PinHeader_2x03_P2.54mm_Vertical, symbol Connector_Generic:Conn_02x03_Odd_Even
- D101: footprint (none) -> Diode_THT:D_DO-35_SOD27_P7.62mm_Horizontal
- J101: footprint Connector_AMASS:AMASS_XT60-M_1x02_P7.20mm_Vertical -> Connector_AMASS:AMASS_XT60PW-M_1x02_P7.20mm_Horizontal
Connections:
- net GND: now also D101.2 (A), C101.2, C102.2, C103.2, C104.2, C105.2, C106.2, C107.2, C108.2
- net VCCF: now also C101.1, C102.1, C103.1, C104.1, C105.1, C106.1, C107.1, C108.1
- net VCC_FUSE: now also J102.1 (Pin_1)
- net at D101.1 (K), K101.A1: now also J102.6 (Pin_6)
- new net: J102.2 (Pin_2), J102.4 (Pin_4)
- new net: J102.3 (Pin_3), J102.5 (Pin_5)
Other:
- moved on the sheet: D101, F101
