File: LV/Outputs.kicad_sch (KiCad schematic)
At the start: 12 parts, among them U201 TPS5460 康威科技, U202 TPS5460 康威科技, U203 TPS5460 康威科技, U204 TPS5460 康威科技

Commit message: added lv
Parts:
- removed C201, C202, C203, C204: 560u, scottcjx-kicad-lib:CP_Radial_D10.0mm_P5.00mm, symbol Device:C_Polarized
- added J201: V_{HV}, Connector_JST:JST_XH_B2B-XH-AM_1x02_P2.50mm_Vertical, symbol Connector_Generic:Conn_01x02
- added J202, J203, J204: V, Connector_PinHeader_2.54mm:PinHeader_2x05_P2.54mm_Vertical, symbol Connector_Generic:Conn_02x05_Odd_Even
- added J205: V_{SBC}, Connector_AMASS:AMASS_XT30UPB-M_1x02_P5.0mm_Vertical, symbol Connector_Generic:Conn_01x02
- C205, C206, C207, C208: footprint scottcjx-kicad-lib:CP_Radial_D10.0mm_P5.00mm -> Capacitor_THT:CP_Radial_D10.0mm_P5.00mm; now not fitted
Connections:
- net +12V: now also J201.1 (Pin_1), J204.1 (Pin_1), J204.3 (Pin_3), J204.5 (Pin_5), J204.7 (Pin_7), J204.9 (Pin_9)
- net +5V: now also J202.1 (Pin_1), J202.3 (Pin_3), J202.5 (Pin_5), J202.7 (Pin_7), J202.9 (Pin_9)
- net +9V: now also J203.1 (Pin_1), J203.3 (Pin_3), J203.5 (Pin_5), J203.7 (Pin_7), J203.9 (Pin_9)
- net GND: now also J201.2 (Pin_2), J202.10 (Pin_10), J202.2 (Pin_2), J202.4 (Pin_4), J202.6 (Pin_6), J202.8 (Pin_8), J203.10 (Pin_10), J203.2 (Pin_2), J203.4 (Pin_4), J203.6 (Pin_6), J203.8 (Pin_8), J204.10 (Pin_10), J204.2 (Pin_2), J204.4 (Pin_4), J204.6 (Pin_6), J204.8 (Pin_8), J205.1 (Pin_1)
- net V_{SBC}: now also J205.2 (Pin_2)
